File: hardware/kicad/x3tuner.kicad_sch (KiCad schematic)
At the start: 53 parts, among them J1 USB-C, J2 AKKU, J3 SWD-ZIEL, Q1 AO3401A, Q2 HJ8205, SW1 EIN/AUS, SW2 RESET, SW3 BOOT, U1 ESP32-S3-WROOM-1-N16R8, U2 TP4056, U3 DW01A, U4 ME6211C33M5G-N, U5 ME6211C33M5G-N, U6 SRV05-4

Commit message: Cost-down rev 1.1: ESP32-C3-WROOM-02 and MSK12C02 switch
Swap the ESP32-S3-WROOM-1-N16R8 for an ESP32-C3-WROOM-02-N4 (about
1.20-1.55 USD less per board at 100+) and the C&K slide switch for an
MSK12C02 (about 0.55 USD less), roughly 30 % off the assembled board.

- new pin plan: SWD on IO5/6/7, sense inputs on ADC1 (IO1/IO3/IO4),
  TGT_EN IO10, LED IO0, BOOT IO9, 10k pull-ups on strapping IO2/IO8
- USB-C moves to the right edge (USB pre-route generalised for either
  orientation), switch to the left; board shrinks to 38 x 54.5 mm
- project footprints: C3 module without 0.2 mm EPAD vias and with a
  board-sized antenna keep-out; MSK12C02 land pattern after the EasyEDA
  footprint for C431540
- re-routed, DRC clean (board and 10-up panel, now 202 x 128 mm)
- case follows the board: side-agnostic ports, 503040 battery bay,
  42 x 65 x 17 mm
- firmware: x3tuner env now targets esp32-c3 with the new pin map
- docs: updated cost tables (about 5.20/4.80/4.50 USD per board at
  100/200/500 incl. VAT), verification notes

Co-Authored-By: Claude Opus 5.5 <noreply@anthropic.com>
Claude-Session: https://claude.ai/code/session_01RVwXhv4cRLa5H5kfiVg79q
Parts:
- added R21, R22: 10k, Resistor_SMD:R_0402_1005Metric, symbol Device:R
- SW1: footprint Button_Switch_SMD:SW_SPDT_CK_JS102011SAQN -> x3tuner:SW_SPDT_MSK12C02; Hersteller C&K -> SHOU HAN; LCSC C221660 -> C431540
- U1: value ESP32-S3-WROOM-1-N16R8 -> ESP32-C3-WROOM-02-N4; footprint x3tuner:ESP32-S3-WROOM-1_JLC -> x3tuner:ESP32-C3-WROOM-02_JLC; symbol RF_Module:ESP32-S3-WROOM-1 -> x3tuner:ESP32-C3-WROOM-02; Beschreibung ESP32-S3, 16 MB Flash, 8 MB Octal-PSRAM -> ESP32-C3, 4 MB Flash, 400 KB SRAM, WiFi + BLE; LCSC C2913202 -> C2934560
Connections:
- net +3V3: now also U1.1 (3V3), R21.1, R22.1; no longer U1.2 (3V3)
- net BOOT: now also U1.8 (IO9); no longer U1.27 (IO0)
- net EN: now also U1.2 (EN); no longer U1.3 (EN)
- net GND: now also U1.19 (EPAD), U1.9 (GND); no longer U1.1 (GND), U1.40 (GND), U1.41 (GND)
- net LED: now also U1.18 (IO0); no longer U1.23 (IO21)
- net NRST: now also U1.6 (IO7); no longer U1.19 (IO11)
- net RXD0: now also U1.11 (RXD/IO20); no longer U1.36 (RXD0)
- net SWCLK: now also U1.4 (IO5); no longer U1.20 (IO12)
- net SWDIO: now also U1.5 (IO6); no longer U1.21 (IO13)
- net TGT_EN: now also U1.10 (IO10); no longer U1.22 (IO14)
- net TXD0: now also U1.12 (TXD/IO21); no longer U1.37 (TXD0)
- net VBAT_SENSE: now also U1.3 (IO4); no longer U1.17 (IO9)
- net VBUS_SENSE: now also U1.17 (IO1); no longer U1.12 (IO8)
- net VTGT_SENSE: now also U1.15 (IO3); no longer U1.38 (IO2)
- net STRAP_IO2: now reaches U1.16 (IO2)
- net STRAP_IO2: now also R22.2
- net STRAP_IO8: now reaches U1.7 (IO8)
- net STRAP_IO8: now also R21.2
- no-connect marks 30 -> 7
Other:
- note added: "ESP32-C3-WROOM-02-N4"
- note added: "IO2/IO8 (Strapping) per 10k auf High, IO9 = BOOT."
- note added: "U5 schaltet die VCU-Versorgung (GPIO10):"
- note removed: "ESP32-S3-WROOM-1-N16R8"
- note removed: "U5 schaltet die VCU-Versorgung (GPIO14):"
- title: X3-Tuner — ESP32-S3 SWD-Programmer mit Akku -> X3-Tuner — ESP32-C3 SWD-Programmer mit Akku

Commit message: Cut JLC assembly cost, assemble every part, price with live JLC data
Checked every BOM line live on jlcpcb.com (price, stock, library type):
- U6: ProTek SRV05-4 (C85364) was out of stock (pre-order, MOQ 30);
  now the pin-identical TECH PUBLIC SRV05-4 (C558418, 219k in stock).
- D4: the yellow LED is an extended part (+$3 fee); now the basic white
  KT-0603W (C2290) with a 100 R series resistor.
- J3: the SWD header is now assembled by JLC as well (C32713264, THT),
  so the board needs no hand soldering at all.

The README cost section now uses the live part prices, the PCB price and
shipping from the JLC quote page, and the official fee schedule (10
extended part types, hand-soldering fee for J3). CPL rotations are
normalised to 0..360.

Co-Authored-By: Claude Opus 5.5 <noreply@anthropic.com>
Claude-Session: https://claude.ai/code/session_01RVwXhv4cRLa5H5kfiVg79q
Parts:
- D4: value yellow -> white; Beschreibung Status-LED gelb -> Status-LED weiß; LCSC C89811 -> C2290
- J3: Hersteller (none) -> hanxia; LCSC (none) -> C32713264
- R20: value 1k -> 100; LCSC C11702 -> C25076
- U6: Hersteller ProTek -> TECH PUBLIC; LCSC C85364 -> C558418
Changed lines of the file:
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@@
     (property "Reference" "R20" (at 301.752 190.5 90)
       (effects (font (size 1.27 1.27))))
-    (property "Value" "1k" (at 299.72 190.5 90)
+    (property "Value" "100" (at 299.72 190.5 90)
       (effects (font (size 1.27 1.27))))
     (property "Footprint" "Resistor_SMD:R_0402_1005Metric" (at 299.72 190.5 0)
@@
     (property "Datasheet" "" (at 299.72 190.5 0)
       (effects (font (size 1.27 1.27)) hide))
-    (property "LCSC" "C11702" (at 299.72 190.5 0)
+    (property "LCSC" "C25076" (at 299.72 190.5 0)
       (effects (font (size 1.27 1.27)) hide))
     (property "Beschreibung" "Status-LED" (at 299.72 190.5 0)
@@
     (property "Reference" "D4" (at 299.72 201.93 0)
       (effects (font (size 1.27 1.27))))
-    (property "Value" "yellow" (at 299.72 207.01 0)
+    (property "Value" "white" (at 299.72 207.01 0)
       (effects (font (size 1.27 1.27))))
     (property "Footprint" "LED_SMD:LED_0603_1608Metric" (at 299.72 204.47 0)
@@
     (property "Datasheet" "" (at 299.72 204.47 0)
       (effects (font (size 1.27 1.27)) hide))
-    (property "LCSC" "C89811" (at 299.72 204.47 0)
-      (effects (font (size 1.27 1.27)) hide))
-    (property "Beschreibung" "Status-LED gelb" (at 299.72 204.47 0)
+    (property "LCSC" "C2290" (at 299.72 204.47 0)
+      (effects (font (size 1.27 1.27)) hide))
+    (property "Beschreibung" "Status-LED weiß" (at 299.72 204.47 0)
       (effects (font (size 1.27 1.27)) hide))
     (pin "1")
@@
     (property "Datasheet" "" (at 85.09 90.17 0)
       (effects (font (size 1.27 1.27)) hide))
-    (property "LCSC" "C85364" (at 85.09 90.17 0)
-      (effects (font (size 1.27 1.27)) hide))
-    (property "Hersteller" "ProTek" (at 85.09 90.17 0)
+    (property "LCSC" "C558418" (at 85.09 90.17 0)
+      (effects (font (size 1.27 1.27)) hide))
+    (property "Hersteller" "TECH PUBLIC" (at 85.09 90.17 0)
       (effects (font (size 1.27 1.27)) hide))
     (property "Beschreibung" "USB ESD-Schutz" (at 85.09 90.17 0)
@@
     (property "Datasheet" "" (at 394.97 95.25 0)
       (effects (font (size 1.27 1.27)) hide))
+    (property "LCSC" "C32713264" (at 394.97 95.25 0)
+      (effects (font (size 1.27 1.27)) hide))
+    (property "Hersteller" "hanxia" (at 394.97 95.25 0)
+      (effects (font (size 1.27 1.27)) hide))
     (property "Beschreibung" "Stiftleiste 1x5 gewinkelt zum Scooter (3V3 DIO CLK RST GND)" (at 394.97 95.25 0)
