File: hardware/carrier/kicad/x3carrier.kicad_sch (KiCad schematic)
At the start: 31 parts, among them J1 Sockel SuperMini, J2 Sockel SuperMini, J3 AKKU, J4 SWD-ZIEL, Q1 AO3401A, Q2 AO3401A, SW1 EIN/AUS, U1 TP4056

Commit message: X3-Tuner Mini as a stick: narrow carrier board and 3D-printed case
Carrier board (Rev 1.1) redesigned as a 20.5 x 65 mm stick: the
SuperMini sits at the front with its USB-C in the end face, the SWD
header at the rear, the charger between the socket rows. New P-MOSFET
Q3 as battery reverse-polarity protection (cheap JST-PH cells often
have swapped leads), charge current lowered to ~235 mA (R1 = 5.1k) for
300-400 mAh cells. Routed, DRC clean; panel and NextPCB rail variant
(12 mm rails, 50.6 x 65 mm) regenerated.

Case: the X3-Tuner case model is now a shared core (case_core.scad)
with one small wrapper per board; the X3-Tuner STLs are unchanged.
New options for the stick: USB-C in the end face, battery pocket under
the lid, ribs pressing the SuperMini into its sockets, windows over its
LEDs/buttons, pin labels above the SWD slot. make_case_data.py and
make_case.sh build either board via X3_CIRCUIT. The Mini case is
77.7 x 24.4 x 22.4 mm for an 802030 LiPo and was checked for collisions
with board, SuperMini and battery.

Co-Authored-By: Claude Opus 5.5 <noreply@anthropic.com>
Claude-Session: https://claude.ai/code/session_01RVwXhv4cRLa5H5kfiVg79q
Parts:
- added Q3: AO3401A, Package_TO_SOT_SMD:SOT-23, symbol Transistor_FET:AO3401A
- J3: Beschreibung LiPo 1S mit Schutzschaltung, JST-PH 2.0 -> LiPo 1S mit Schutzschaltung, JST-PH 2.0, + = Pin 1
- R1: value 3.3k -> 5.1k; Beschreibung PROG: I = 1200/R ≈ 364 mA -> PROG: I = 1200/R ≈ 235 mA; LCSC C25890 -> C25905
- U1: Beschreibung Li-Ion Lader 1S, ~360 mA -> Li-Ion Lader 1S, ~235 mA
Connections:
- net GND: now also Q3.1 (G)
- net VBAT: now also Q3.2 (S); no longer J3.1 (Pin_1)
- new net BAT_IN: J3.1 (Pin_1), Q3.3 (D)
Other:
- note added: "Akku 1S LiPo (mit Schutz) + Verpolschutz + Ein/Aus"
- note added: "Akkubetrieb: Akku -> Q3 -> Q1 (Schalter) -> D1 -> 5V-Pin."
- note added: "Ladestrom R1 = 5,1k -> ca. 235 mA."
- note added: "Q3 = Verpolschutz: leitet nur mit + an Pin 1."
- note removed: "Akku 1S LiPo (mit Schutz) + Ein/Aus"
- note removed: "Akkubetrieb: Akku -> Q1 (Schalter) -> D1 -> 5V-Pin."
- note removed: "Ladestrom R1 = 3,3k -> ca. 360 mA."

Commit message: X3-Tuner Mini Rev 1.2: pin headers, closed case, Wi-Fi OTA + flash lock
The ESP32-C3 SuperMini has no pins, so the carrier now carries two 1x8
male headers (factory-soldered); the module is pushed on and clamped by
the lid. Same pads/routing as the sockets, DRC clean; panel and NextPCB
variant regenerated. The header's LCSC number could not be verified
(jlcpcb.com unreachable) and is left blank in the BOM; make_fab/make_panel
now keep LCSC-less parts in the BOM/CPL and warn, instead of silently
dropping them.

Case: no openings over the SuperMini — RESET/BOOT are unreachable and the
module is fully enclosed. The module sits flat on the headers (not on tall
sockets), so the case is driven by the lid battery and drops to 20.9 mm.
Battery pocket now for a 6-7 mm cell (clears the JST socket); the clamp is
split into two ribs that avoid the chip antenna. Collision-checked against
board, SuperMini and battery.

Firmware: Wi-Fi OTA endpoint (src/ota.h, POST /api/ota) on the x3carrier
build with an OTA-capable partition, so the app can update the device with
USB download mode locked. hardware/carrier/SECURITY.md documents the
one-time eFuse hardening (flash encryption, Secure Boot v2, disabling the
download mode) that makes the firmware non-readable and non-flashable while
keeping signed OTA updates.

Co-Authored-By: Claude Opus 4.8 <noreply@anthropic.com>
Claude-Session: https://claude.ai/code/session_01RVwXhv4cRLa5H5kfiVg79q
Parts:
- J1, J2: value Sockel SuperMini -> Stift SuperMini; footprint Connector_PinSocket_2.54mm:PinSocket_1x08_P2.54mm_Vertical -> Connector_PinHeader_2.54mm:PinHeader_1x08_P2.54mm_Vertical; Beschreibung Buchsenleiste 1x8 2,54 mm (H 8,5 mm) fuer ESP32-C3 SuperMini -> Stiftleiste 1x8 2,54 mm fuer ESP32-C3 SuperMini (aufgesteck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; LCSC C42431840 -> (none)
Changed lines of the file:
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@@
     (title "X3-Tuner Mini — Traeger fuer ESP32-C3 SuperMini")
     (date "2026-10-05")
-    (rev "1.1")
+    (rev "1.2")
     (company "x3utils-esp32")
     (comment 1 "Generiert aus hardware/gen/circuit_carrier.py - nicht von Hand editieren, sondern circuit_carrier.py aendern")
@@
     (property "Reference" "J1" (at 59.69 49.53 0)
       (effects (font (size 1.27 1.27))))
-    (property "Value" "Sockel SuperMini" (at 59.69 72.39 0)
+    (property "Value" "Stift SuperMini" (at 59.69 72.39 0)
       (effects (font (size 1.27 1.27))))
-    (property "Footprint" "Connector_PinSocket_2.54mm:PinSocket_1x08_P2.54mm_Vertical" (at 59.69 59.69 0)
+    (property "Footprint" "Connector_PinHeader_2.54mm:PinHeader_1x08_P2.54mm_Vertical" (at 59.69 59.69 0)
       (effects (font (size 1.27 1.27)) hide))
     (property "Datasheet" "" (at 59.69 59.69 0)
       (effects (font (size 1.27 1.27)) hide))
-    (property "LCSC" "C42431840" (at 59.69 59.69 0)
-      (effects (font (size 1.27 1.27)) hide))
-    (property "Beschreibung" "Buchsenleiste 1x8 2,54 mm (H 8,5 mm) fuer ESP32-C3 SuperMini" (at 59.69 59.69 0)
+    (property "Beschreibung" "Stiftleiste 1x8 2,54 mm fuer ESP32-C3 SuperMini (aufgesteckt)" (at 59.69 59.69 0)
       (effects (font (size 1.27 1.27)) hide))
     (pin "1")
@@
     (property "Reference" "J2" (at 59.69 100.33 0)
       (effects (font (size 1.27 1.27))))
-    (property "Value" "Sockel SuperMini" (at 59.69 123.19 0)
+    (property "Value" "Stift SuperMini" (at 59.69 123.19 0)
       (effects (font (size 1.27 1.27))))
-    (property "Footprint" "Connector_PinSocket_2.54mm:PinSocket_1x08_P2.54mm_Vertical" (at 59.69 110.49 0)
+    (property "Footprint" "Connector_PinHeader_2.54mm:PinHeader_1x08_P2.54mm_Vertical" (at 59.69 110.49 0)
       (effects (font (size 1.27 1.27)) hide))
     (property "Datasheet" "" (at 59.69 110.49 0)
       (effects (font (size 1.27 1.27)) hide))
-    (property "LCSC" "C42431840" (at 59.69 110.49 0)
-      (effects (font (size 1.27 1.27)) hide))
-    (property "Beschreibung" "Buchsenleiste 1x8 2,54 mm (H 8,5 mm) fuer ESP32-C3 SuperMini" (at 59.69 110.49 0)
+    (property "Beschreibung" "Stiftleiste 1x8 2,54 mm fuer ESP32-C3 SuperMini (aufgesteckt)" (at 59.69 110.49 0)
       (effects (font (size 1.27 1.27)) hide))
     (pin "1")
